File: NoBootLoadFlasher_QFP32toDIP28/NoBootLoadFlasher.kicad_pcb (KiCad board)
At the start: 2 copper layers, 45.8 x 100.5 mm, 9 parts

Commit message: Add files via upload
Routing:
- net GND: vias 27 -> 29
Other:
- board text added: "LGT8F328P BARE IC FLASHING"
- board text removed: "LTG8F328P BARE IC FLASHING"
Changed lines of the file:
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@@
     (effects (font (size 1 1) (thickness 0.1)) (justify left bottom))
   )
-  (gr_text "LTG8F328P BARE IC FLASHING" (at 74.1934 171.6024) (layer "F.SilkS")
+  (gr_text "LGT8F328P BARE IC FLASHING" (at 74.1934 171.6024) (layer "F.SilkS")
     (effects (font (size 1.5 1.5) (thickness 0.3) bold) (justify left bottom))
   )
@@
     )
   )
+  (via (at 102.87 83.82) (size 0.6) (drill 0.3) (layers "F.Cu" "B.Cu") (free) (net 1))
   (via (at 95.25 117.221) (size 0.6) (drill 0.3) (layers "F.Cu" "B.Cu") (free) (net 1))
+  (via (at 99.06 83.82) (size 0.6) (drill 0.3) (layers "F.Cu" "B.Cu") (free) (net 1))
   (via (at 87.122 114.681) (size 0.6) (drill 0.3) (layers "F.Cu" "B.Cu") (free) (net 1))
   (via (at 108.839 136.017) (size 0.6) (drill 0.3) (layers "F.Cu" "B.Cu") (free) (net 1))
